File: PCB Design/Digi2_Act8085.kicad_sch (KiCad schematic)
At the start: 20 parts, among them U1 8085A, U2 Barrel_Jack, U3 L7805, Y1 3MHz

Commit message: newwwwwwwwww
Parts:
- C12: footprint Capacitor_THT:CP_Radial_D8.0mm_P3.50mm -> Capacitor_THT:CP_Radial_D5.0mm_P2.50mm
Changed lines of the file:
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@@
 			)
 		)
-		(property "Footprint" "Capacitor_THT:CP_Radial_D8.0mm_P3.50mm"
+		(property "Footprint" "Capacitor_THT:CP_Radial_D5.0mm_P2.50mm"
 			(at 43.18 127 0)
 			(effects
