File: PCB Design/Digi2_Act8085.kicad_pcb (KiCad board)
At the start: 2 copper layers, 27 parts, among them U1 8085A, U10 8255, U2 Barrel_Jack, U3 L7805, U4 2764, U5 CY6264, U6 74LS373, U7 74LS138, U8 8255, U9 8255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

Commit message: copy of main(1)
Parts:
- moved C1 5.86 mm to (165.5, 64.5)
- moved C10 5.86 mm to (166.8, 49.5)
- moved C11 5.86 mm to (166.8, 55.5)
- moved D1 5.86 mm to (149.0, 54.7)
- moved D2 5.86 mm to (159.0, 41.6)
- moved FB1 5.86 mm to (166.8, 44.8)
- moved R1 5.86 mm to (152.2, 48.6)
- moved U2 5.86 mm to (157.0, 36.8)
- moved U3 5.86 mm to (159.0, 64.1)

Commit message: test merge D
Parts:
- moved C1 5.86 mm to (161.0, 68.2)
- moved C10 5.86 mm to (162.2, 53.2)
- moved C11 5.86 mm to (162.2, 59.2)
- moved D1 5.86 mm to (144.5, 58.5)
- moved D2 5.86 mm to (154.5, 45.4)
- moved FB1 5.86 mm to (162.2, 48.5)
- moved R1 5.86 mm to (147.8, 52.3)
- moved U2 5.86 mm to (152.5, 40.5)
- moved U3 5.86 mm to (154.5, 67.8)
Routing:
- net Net-(C12-+): track 0.00 -> 7.42 mm

Commit message: test merge3
Parts:
- moved C1 3.79 mm to (157.3, 67.7)
- moved D1 3.79 mm to (140.8, 57.9)
- moved U3 3.79 mm to (150.8, 67.3)
- moved C10 3.79 mm to (158.5, 52.7)
- moved C11 3.79 mm to (158.5, 58.7)
- moved D2 3.79 mm to (150.8, 44.8)
- moved FB1 3.79 mm to (158.5, 48.0)
- moved R1 3.79 mm to (144.0, 51.8)
- moved U2 3.79 mm to (148.8, 40.0)
Routing:
- net GND: track 78.0 -> 107.8 mm
