File: PCB Design/Memory.kicad_sch (KiCad schematic)
At the start: 2 parts, among them U4 2764, U5 CY6264

Commit message: newwwwwwwwww
Parts:
- U5: footprint Package_DIP:DIP-28_W15.24mm_Socket -> Package_DIP:DIP-28_W15.24mm
Changed lines of the file:
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@@
 			)
 		)
-		(property "Footprint" "Package_DIP:DIP-28_W15.24mm_Socket"
+		(property "Footprint" "Package_DIP:DIP-28_W15.24mm"
 			(at 177.8 51.816 0)
 			(effects
