File: PCB Design/Memory_PPI.kicad_sch (KiCad schematic)
At the start: 2 parts, among them U6 74LS373, U7 74LS138

Commit message: newwwwwwwwww
Parts:
- U6: footprint Package_DIP:DIP-20_W7.62mm_Socket -> Package_DIP:DIP-20_W7.62mm
- U7: footprint Package_DIP:DIP-16_W7.62mm_Socket -> Package_DIP:DIP-16_W7.62mm
Changed lines of the file:
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@@
 			)
 		)
-		(property "Footprint" "Package_DIP:DIP-16_W7.62mm_Socket"
+		(property "Footprint" "Package_DIP:DIP-16_W7.62mm"
 			(at 92.71 124.46 0)
 			(effects
@@
 			)
 		)
-		(property "Footprint" "Package_DIP:DIP-20_W7.62mm_Socket"
+		(property "Footprint" "Package_DIP:DIP-20_W7.62mm"
 			(at 88.9 54.61 0)
 			(effects
